File: keyboard/pcb/arrak_keyboard.kicad_pcb (KiCad board)
At the start: 2 copper layers, 40 parts, among them J1 Conn_01x18_Male, J2 Conn_01x18_Male, J3 Conn_01x02_Male, J4 Conn_01x02_Male, SW1 SW_PUSH, SW10 SW_PUSH, SW11 SW_PUSH, SW12 SW_PUSH, SW13 SW_PUSH, SW14 SW_PUSH, SW15 SW_PUSH, SW16 SW_PUSH, SW17 SW_PUSH, SW18 SW_PUSH, SW19 SW_PUSH, SW2 SW_PUSH, SW20 SW_PUSH, SW21 SW_PUSH, SW22 SW_PUSH, SW23 SW_PUSH, SW24 SW_PUSH, SW25 SW_PUSH, SW26 SW_PUSH, SW27 SW_PUSH, SW28 SW_PUSH, SW29 SW_PUSH, SW3 SW_PUSH, SW30 SW_PUSH, SW31 SW_PUSH, SW32 SW_PUSH, SW33 SW_PUSH, SW34 SW_PUSH, SW35 SW_PUSH, SW36 SW_PUSH, SW4 SW_PUSH, SW5 SW_PUSH, SW6 SW_PUSH, SW7 SW_PUSH, SW8 SW_PUSH, SW9 SW_PUSH

Commit message: placement of switch footprints complete
Parts:
- moved J4 189.2 mm to (257.6, 51.3)
- moved J2 171.2 mm to (236.0, 16.4)
- moved SW36 153.1 mm to (294.1, 178.2)
- moved SW22 152.3 mm to (338.3, 93.0)
- moved SW23 152.3 mm to (342.7, 109.5)
- moved SW24 152.3 mm to (347.1, 125.9)
- moved SW19 152.3 mm to (360.8, 107.7)
- moved SW20 152.3 mm to (365.2, 124.1)
- moved SW21 152.3 mm to (369.6, 140.6)
- moved SW29 152.3 mm to (304.8, 107.2)
- moved SW30 152.3 mm to (309.2, 123.6)
- moved SW31 152.3 mm to (313.6, 140.0)
- moved SW33 152.3 mm to (287.9, 113.8)
- moved SW34 152.3 mm to (292.3, 130.2)
- moved SW25 152.3 mm to (319.3, 91.9)
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Other:
- board outline added: 103.6 x 75.9 mm

Commit message: finish physical layout of keyboard?
Parts:
- moved J2 97.9 mm to (257.9, 111.8), turned to 255 degrees
- moved J1 94.6 mm to (156.9, 111.8), turned to 105 degrees
- moved J3 67.9 mm to (145.9, 114.8), turned to 180 degrees
- moved J4 64.5 mm to (268.9, 114.8), turned to 180 degrees
Other:
- board size 103.6 x 75.9 mm -> 346.3 x 109.3 mm

Commit message: weird routing
Parts:
- SW1, SW10, SW11, SW12, SW13, SW14, SW15, SW16, SW17, SW18, SW19, SW2, SW20, SW21, SW22, SW23, SW24, SW25, SW26, SW27, SW28, SW29, SW3, SW30, SW31, SW32, SW33, SW34, SW35, SW36, SW4, SW5, SW6, SW7, SW8, SW9: footprint Keebio-Parts:Kailh-PG1350-1u-reversible-NoLED -> Keebio-Parts:Kailh-PG1350-1u-NoLED
- moved SW22 95.9 mm to (294.1, 178.2), turned to 45 degrees
- moved SW36 84.4 mm to (369.6, 140.6), turned to 15 degrees
- moved SW19 73.2 mm to (287.9, 113.8)
- moved SW20 73.2 mm to (292.3, 130.2)
- moved SW21 73.2 mm to (296.7, 146.6)
- moved SW34 72.1 mm to (360.8, 107.7)
- moved SW35 72.1 mm to (365.2, 124.1)
- moved SW32 65.1 mm to (342.7, 109.5), turned to 15 degrees
- moved SW33 60.4 mm to (347.1, 125.9)
- moved SW26 59.1 mm to (310.2, 165.8), turned to 30 degrees
- moved SW31 53.1 mm to (338.3, 93.0)
- moved SW28 50.0 mm to (323.7, 108.3)
- moved SW25 48.8 mm to (313.6, 140.4)
- moved SW30 39.7 mm to (328.9, 158.1)
- moved SW23 37.9 mm to (304.8, 107.2)
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Connections:
- J1 pad 1: D18 -> D3
- J1 pad 10: D9 -> D12
- J1 pad 12: D7 -> D5
- J1 pad 13: D6 -> D2
- J1 pad 14: D5 -> D15
- J1 pad 15: D4 -> D11
- J1 pad 16: D3 -> D7
- J1 pad 17: D2 -> D4
- J1 pad 2: D17 -> D6
- J1 pad 4: D15 -> D9
- J1 pad 5: D14 -> D13
- J1 pad 6: D13 -> D17
- J1 pad 7: D12 -> D10
- J1 pad 8: D11 -> D14
- J1 pad 9: D10 -> D18
- J2 pad 10: D27 -> D20
- J2 pad 14: D23 -> D19
- J2 pad 15: D22 -> D23
- J2 pad 16: D21 -> D27
- J2 pad 17: D20 -> D31
- J2 pad 18: D19 -> D34
- J2 pad 3: D34 -> D22
- J2 pad 6: D31 -> D21
- SW19 pad 2: D33 -> D19
- SW20 pad 2: D34 -> D20
- SW21 pad 2: D35 -> D21
- SW22 pad 2: D36 -> D22
- SW23 pad 2: D29 -> D23
- SW24 pad 2: D30 -> D24
- SW25 pad 2: D31 -> D25
- SW26 pad 2: D32 -> D26
- SW27 pad 2: D25 -> D27
- SW28 pad 2: D26 -> D28
- SW29 pad 2: D27 -> D29
- SW30 pad 2: D28 -> D30
- SW31 pad 2: D22 -> D31
- SW32 pad 2: D23 -> D32
- SW33 pad 2: D24 -> D33
- SW34 pad 2: D19 -> D34
- SW35 pad 2: D20 -> D35
- SW36 pad 2: D21 -> D36
Routing:
- net R3: track 0.00 -> 318.7 mm
- net R4: track 0.00 -> 277.9 mm
- net R2: track 0.00 -> 216.7 mm
- net R1: track 0.00 -> 208.5 mm
- net D1: track 0.00 -> 180.1 mm
- net D34: track 0.00 -> 170.3 mm
- net D2: track 0.00 -> 165.2 mm
- net D4: track 0.00 -> 149.1 mm
- net D18: track 0.00 -> 143.4 mm
- net D3: track 0.00 -> 139.8 mm
- net D5: track 0.00 -> 133.7 mm
- net D10: track 0.00 -> 126.1 mm
- net D14: track 0.00 -> 125.5 mm
- net D7: track 0.00 -> 122.6 mm
- net D6: track 0.00 -> 113.8 mm
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
Commit message: lite bättre routing
Parts:
- removed J3, J4: Conn_01x02_Male, Connector_PinSocket_2.54mm:PinSocket_1x02_P2.54mm_Vertical
- J1, J2: value Conn_01x18_Male -> Conn_01x20_Male; footprint Connector_PinHeader_2.54mm:PinHeader_1x18_P2.54mm_Vertical -> Connector_PinHeader_2.54mm:PinHeader_1x20_P2.54mm_Vertical
- moved SW11 27.0 mm to (97.0, 83.6)
- moved SW4 27.0 mm to (63.5, 69.5)
- moved SW21 27.0 mm to (283.7, 123.0)
- moved SW28 27.0 mm to (310.7, 84.7)
- moved SW19 27.0 mm to (274.9, 90.2)
- moved SW23 27.0 mm to (291.7, 83.6)
- moved SW26 27.0 mm to (297.1, 142.2)
- moved SW30 27.0 mm to (315.8, 134.5)
- moved SW8 27.0 mm to (78.1, 84.7)
- moved SW35 27.0 mm to (352.2, 100.5)
- moved SW7 27.0 mm to (82.5, 68.3)
- moved J2 27.0 mm to (244.9, 88.2)
- moved SW20 27.0 mm to (279.3, 106.6)
- moved SW9 27.0 mm to (73.7, 101.2)
- moved J1 27.0 mm to (143.9, 88.2)
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Connections:
- J1 pad 2: D6 -> D16
- J1 pad 3: D16 -> D6
- J2 pad 10: D20 -> D24
- J2 pad 11: D26 -> D28
- J2 pad 12: D25 -> D32
- J2 pad 13: D24 -> D35
- J2 pad 2: D35 -> D33
- J2 pad 3: D22 -> D29
- J2 pad 4: D33 -> D25
- J2 pad 5: D32 -> D20
- J2 pad 8: D29 -> D26
- J2 pad 9: D28 -> D22
Routing:
- net R1: track 208.5 -> 399.2 mm
- net R2: track 216.7 -> 396.9 mm
- net D35: track 0.00 -> 166.6 mm
- net D22: track 0.00 -> 157.5 mm
- net D36: track 0.00 -> 138.9 mm
- net D26: track 0.00 -> 134.0 mm
- net D32: track 0.00 -> 128.9 mm
- net D30: track 0.00 -> 122.1 mm
- net R4: track 277.9 -> 395.2 mm, vias 0 -> 2
- net R3: track 318.7 -> 432.1 mm, vias 0 -> 1
- net D33: track 0.00 -> 105.8 mm
- net D27: track 0.00 -> 100.2 mm
- net D28: track 0.00 -> 94.6 mm
- net D29: track 0.00 -> 86.9 mm
- net D24: track 0.00 -> 85.7 mm
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Other:
- outline, holes or cut-outs redrawn

Commit message: finish keyboard pcb
Parts:
- moved SW28 28.6 mm to (308.4, 113.3)
- moved SW6 28.6 mm to (52.4, 130.8)
- moved SW30 28.6 mm to (313.6, 163.0)
- moved SW5 28.6 mm to (56.8, 114.4)
- moved SW7 28.6 mm to (80.2, 96.9)
- moved SW8 28.6 mm to (75.8, 113.3)
- moved SW26 28.6 mm to (294.8, 170.8)
- moved SW1 28.6 mm to (38.7, 112.7)
- moved SW12 28.6 mm to (90.3, 128.6)
- moved SW4 28.6 mm to (61.2, 98.0)
- moved SW18 28.6 mm to (105.5, 183.1)
- moved SW21 28.6 mm to (281.4, 151.6)
- moved SW31 28.6 mm to (322.9, 98.0)
- moved SW22 28.6 mm to (278.7, 183.1)
- moved SW3 28.6 mm to (29.9, 145.5)
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Connections:
- J1 pad 1: D3 -> D15
- J1 pad 10: D12 -> D9
- J1 pad 12: D5 -> D7
- J1 pad 13: D2 -> D6
- J1 pad 14: D15 -> D5
- J1 pad 15: D11 -> D4
- J1 pad 16: D7 -> D3
- J1 pad 17: D4 -> D2
- J1 pad 3: D6 -> D17
- J1 pad 4: D9 -> D18
- J1 pad 5: D13 -> D11
- J1 pad 6: D17 -> D12
- J1 pad 7: D10 -> D13
- J1 pad 9: D18 -> D10
- J2 pad 1: D36 -> D19
- J2 pad 10: D24 -> D29
- J2 pad 12: D32 -> D27
- J2 pad 13: D35 -> D33
- J2 pad 14: D19 -> D32
- J2 pad 15: D23 -> D31
- J2 pad 16: D27 -> D36
- J2 pad 17: D31 -> D35
- J2 pad 2: D33 -> D20
- J2 pad 3: D29 -> D21
- J2 pad 4: D25 -> D22
- J2 pad 5: D20 -> D23
- J2 pad 6: D21 -> D24
- J2 pad 7: D30 -> D25
- J2 pad 9: D22 -> D30
Routing:
- net D3: track 141.0 -> 223.2 mm
- net D36: track 138.9 -> 213.1 mm
- net D6: track 117.6 -> 174.3 mm
- net R3: track 432.1 -> 486.9 mm, vias 1 -> 2
- net D19: track 70.5 -> 30.1 mm, vias 1 -> 0
- net D23: track 84.6 -> 123.8 mm
- net D33: track 105.8 -> 144.3 mm
- net D11: track 95.7 -> 132.9 mm
- net R4: track 395.2 -> 430.3 mm, vias 2 -> 4
- net D35: track 166.6 -> 200.2 mm
- net D2: track 177.4 -> 209.5 mm
- net D24: track 85.7 -> 115.0 mm
- net D29: track 86.9 -> 114.6 mm
- net D25: track 75.9 -> 102.3 mm
- net D12: track 95.1 -> 121.3 mm
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
Commit message: routing on wf module done
Parts:
- added BT1: Battery_Cell, Battery:BatteryHolder_Keystone_3034_1x20mm, B.Cu at (173.6, 114.4)
- added J3: Conn_01x20_Male, Connector_PinHeader_2.54mm:PinHeader_1x20_P2.54mm_Vertical, F.Cu at (225.6, 116.8)
- added J4: Conn_01x20_Male, Connector_PinHeader_2.54mm:PinHeader_1x20_P2.54mm_Vertical, F.Cu at (127.4, 90.5)
- added U1: core51822b_Core51822B, redox_w_footprints:MY-YJ-14015-Module, F.Cu at (183.4, 77.8)
- moved SW19 50.4 mm to (279.4, 168.6)
- moved SW27 50.4 mm to (310.8, 146.8)
- moved SW28 50.4 mm to (315.2, 163.2)
- moved SW29 50.4 mm to (319.6, 179.6)
- moved J2 50.4 mm to (249.8, 165.3)
- moved SW1 50.4 mm to (45.5, 162.6)
- moved SW20 50.4 mm to (283.8, 185.1)
- moved SW21 50.4 mm to (288.2, 201.5)
- moved SW22 50.4 mm to (285.6, 233.0)
- moved SW24 50.4 mm to (300.7, 178.5)
- moved SW25 50.4 mm to (305.1, 195.2)
- moved SW26 50.4 mm to (301.7, 220.7)
- moved SW4 50.4 mm to (68.1, 147.9)
- moved SW8 50.4 mm to (82.6, 163.2)
- moved J1 50.4 mm to (148.1, 165.3)
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Routing:
- net VCC: track 0.00 -> 73.2 mm, vias 0 -> 3
- net GND: track 0.00 -> 62.0 mm, vias 0 -> 1
- net C5: track 0.00 -> 59.8 mm
- net C6: track 0.00 -> 59.8 mm
- net C7: track 0.00 -> 50.6 mm
- net C4: track 0.00 -> 50.6 mm
- net C3: track 0.00 -> 41.5 mm
- net C8: track 0.00 -> 41.5 mm
- net C2: track 0.00 -> 32.3 mm
- net C9: track 0.00 -> 32.3 mm
- net R1u: track 0.00 -> 28.4 mm, vias 0 -> 1
- net C1: track 0.00 -> 25.7 mm
- net C10: track 0.00 -> 25.7 mm
- net R3u: track 0.00 -> 19.4 mm, vias 0 -> 1
- net R4u: track 0.00 -> 15.2 mm, vias 0 -> 1
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Other:
- board size 346.3 x 109.3 mm -> 346.3 x 162.2 mm
